File: windNumber/windNumber.kicad_sch (KiCad schematic)
At the start: 43 parts, among them SW1 SW_Push_45deg, SW10 SW_Push_45deg, SW11 SW_Push_45deg, SW12 SW_Push_45deg, SW13 SW_Push_45deg, SW14 SW_Push_45deg, SW15 SW_Push_45deg, SW16 SW_Push_45deg, SW17 SW_Push_45deg, SW18 SW_Push_45deg, SW19 SW_Push_45deg, SW2 SW_Push_45deg, SW20 SW_Push_45deg, SW21 SW_Push_45deg, SW3 SW_Push_45deg, SW4 SW_Push_45deg, SW5 SW_Push_45deg, SW6 SW_Push_45deg, SW7 SW_Push_45deg, SW8 SW_Push_45deg, SW9 SW_Push_45deg, U1 RP2040_Zero

Commit message: pcb
Parts:
- added D22, D23, D24, D25, D26, D27, D28, D29, D30, D31, D32, D33, D34, D35, D36, D37, D38, D39, D40, D41, D42, D43, D44, D45: LED_SK6812MINI, ScottoKeebs_Components:LED_SK6812MINI, symbol ScottoKeebs:LED_SK6812MINI
Connections:
- net led: now reaches U1.20 (29)
- net led: now also D22.4 (DIN)
- net GND: now reaches U1.22 (GND)
- net GND: now also D22.3 (VSS), D23.3 (VSS), D24.3 (VSS), D25.3 (VSS), D26.3 (VSS), D27.3 (VSS), D28.3 (VSS), D29.3 (VSS), D30.3 (VSS), D31.3 (VSS), D32.3 (VSS), D33.3 (VSS), D34.3 (VSS), D35.3 (VSS), D36.3 (VSS), D37.3 (VSS), D38.3 (VSS), D39.3 (VSS), D40.3 (VSS), D41.3 (VSS), D42.3 (VSS), D43.3 (VSS), D44.3 (VSS), D45.3 (VSS)
- net +5V: now reaches U1.23 (5V)
- net +5V: now also D22.1 (VDD), D23.1 (VDD), D24.1 (VDD), D25.1 (VDD), D26.1 (VDD), D27.1 (VDD), D28.1 (VDD), D29.1 (VDD), D30.1 (VDD), D31.1 (VDD), D32.1 (VDD), D33.1 (VDD), D34.1 (VDD), D35.1 (VDD), D36.1 (VDD), D37.1 (VDD), D38.1 (VDD), D39.1 (VDD), D40.1 (VDD), D41.1 (VDD), D42.1 (VDD), D43.1 (VDD), D44.1 (VDD), D45.1 (VDD)
- new net: D39.2 (DOUT), D40.4 (DIN)
- new net: D38.2 (DOUT), D39.4 (DIN)
- new net: D22.2 (DOUT), D23.4 (DIN)
- new net: D36.2 (DOUT), D37.4 (DIN)
- new net: D35.2 (DOUT), D36.4 (DIN)
- new net: D44.2 (DOUT), D45.4 (DIN)
- new net: D43.2 (DOUT), D44.4 (DIN)
- new net: D26.2 (DOUT), D27.4 (DIN)
- new net: D25.2 (DOUT), D26.4 (DIN)
- new net: D34.2 (DOUT), D35.4 (DIN)
- new net: D33.2 (DOUT), D34.4 (DIN)
- new net: D30.2 (DOUT), D31.4 (DIN)
- new net: D29.2 (DOUT), D30.4 (DIN)
- new net: D41.2 (DOUT), D42.4 (DIN)
- new net: D40.2 (DOUT), D41.4 (DIN)
- new net: D24.2 (DOUT), D25.4 (DIN)
- new net: D23.2 (DOUT), D24.4 (DIN)
- new net: D28.2 (DOUT), D29.4 (DIN)
- new net: D27.2 (DOUT), D28.4 (DIN)
- new net: D31.2 (DOUT), D32.4 (DIN)
- new net: D32.2 (DOUT), D33.4 (DIN)
- new net: D37.2 (DOUT), D38.4 (DIN)
- new net: D42.2 (DOUT), D43.4 (DIN)
