File: windNumber/windNumber.kicad_pcb (KiCad board)
At the start: 2 copper layers, 78 x 120.1 mm, 46 parts, among them SW1 SW_Push_45deg, SW10 SW_Push_45deg, SW11 SW_Push_45deg, SW12 SW_Push_45deg, SW13 SW_Push_45deg, SW14 SW_Push_45deg, SW15 SW_Push_45deg, SW16 SW_Push_45deg, SW17 SW_Push_45deg, SW18 SW_Push_45deg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

Commit message: pcb
Connections:
- U1 pad 20: unconnected-(U1-29-Pad20) -> led
- U1 pad 22: unconnected-(U1-GND-Pad22) -> GND
- U1 pad 23: unconnected-(U1-5V-Pad23) -> +5V
Other:
- board text added: "NumPad"
- board text added: "wind"

Commit message: pcb stuff
Other:
- board text added: "Made by Vejas, 2025"
